File: VintageRadio.kicad_sch (KiCad schematic)
At the start: 26 parts, among them J1 Potmeter, J10 Conn_01x05_Pin, J11 Conn_01x09_Pin, J12 Conn_01x08_Socket, J13 Conn_01x08_Socket, J2 PWR, J3 Out R, J4 Speakers, J5 Volume, J6 Out L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

Commit message: better component placement
Parts:
- removed H3, H4: MountingHole, MountingHole:MountingHole_2mm, symbol Mechanical:MountingHole
- J7: footprint Connector_PinHeader_2.54mm:PinHeader_1x02_P2.54mm_Vertical -> Connector_PinSocket_2.54mm:PinSocket_1x02_P2.54mm_Vertical
Connections:
- net at J6.1 (Pin_1): now also J4.3 (Pin_3); no longer J4.4 (Pin_4)
- net at J6.2 (Pin_2): now also J4.4 (Pin_4); no longer J4.3 (Pin_3)
Other:
- moved on the sheet: H1, H2
Changed lines of the file:
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@@
-	(wire
-		(pts
-			(xy 111.76 90.17) (xy 111.76 33.02)
-		)
-		(stroke
-			(width 0)
-			(type default)
-		)
-	)
 	(wire
 		(pts
@@
 	(wire
 		(pts
+			(xy 121.92 90.17) (xy 114.3 90.17)
+		)
+		(stroke
+			(width 0)
+			(type default)
+		)
+	)
+	(wire
+		(pts
 			(xy 119.38 44.45) (xy 101.6 44.45)
 		)
@@
 	(wire
 		(pts
-			(xy 121.92 90.17) (xy 111.76 90.17)
-		)
-		(stroke
-			(width 0)
-			(type default)
-		)
-	)
-	(wire
-		(pts
 			(xy 152.4 76.2) (xy 152.4 73.66)
 		)
@@
 	(wire
 		(pts
+			(xy 119.38 92.71) (xy 119.38 87.63)
+		)
+		(stroke
+			(width 0)
+			(type default)
+		)
+	)
+	(wire
+		(pts
 			(xy 210.82 140.97) (xy 210.82 99.06)
 		)
@@
 	(wire
 		(pts
-			(xy 114.3 87.63) (xy 114.3 33.02)
-		)
-		(stroke
-			(width 0)
-			(type default)
-		)
-	)
-	(wire
-		(pts
 			(xy 228.6 46.99) (xy 228.6 123.19)
 		)
@@
 	(wire
 		(pts
+			(xy 111.76 33.02) (xy 111.76 92.71)
+		)
+		(stroke
+			(width 0)
+			(type default)
+		)
+	)
+	(wire
+		(pts
 			(xy 165.1 63.5) (xy 165.1 66.04)
 		)
@@
 	(wire
 		(pts
-			(xy 119.38 87.63) (xy 114.3 87.63)
-		)
-		(stroke
-			(width 0)
-			(type default)
-		)
-	)
-	(wire
-		(pts
 			(xy 101.6 57.15) (xy 101.6 44.45)
 		)
@@
 	(wire
 		(pts
+			(xy 111.76 92.71) (xy 119.38 92.71)
+		)
+		(stroke
+			(width 0)
+			(type default)
+		)
+	)
+	(wire
+		(pts
 			(xy 172.72 41.91) (xy 172.72 85.09)
 		)
@@
 		(pts
 			(xy 208.28 138.43) (xy 208.28 101.6)
+		)
+		(stroke
+			(width 0)
+			(type default)
+		)
+	)
+	(wire
+		(pts
+			(xy 114.3 33.02) (xy 114.3 90.17)
 		)
 		(stroke
@@
 			)
 		)
-		(property "Footprint" "Connector_PinHeader_2.54mm:PinHeader_1x02_P2.54mm_Vertical"
+		(property "Footprint" "Connector_PinSocket_2.54mm:PinSocket_1x02_P2.54mm_Vertical"
 			(at 142.24 25.4 0)
 			(effects
@@
 	(symbol
 		(lib_id "Mechanical:MountingHole")
-		(at 266.7 143.51 0)
+		(at 261.62 160.02 0)
+		(mirror y)
 		(unit 1)
 		(exclude_from_sim yes)
@@
 		(on_board yes)
 		(dnp no)
-		(fields_autoplaced yes)
 		(property "Reference" "H1"
-			(at 269.24 142.2399 0)
+			(at 259.08 158.7499 0)
 			(effects
 				(font
@@
 		)
 		(property "Value" "MountingHole"
-			(at 269.24 144.7799 0)
+			(at 259.08 161.2899 0)
 			(effects
 				(font
@@
 		)
 		(property "Footprint" "MountingHole:MountingHole_2mm"
-			(at 266.7 143.51 0)
+			(at 261.62 160.02 0)
 			(effects
 				(font
@@
 		)
 		(property "Datasheet" "~"
-			(at 266.7 143.51 0)
+			(at 261.62 160.02 0)
 			(effects
 				(font
@@
 		)
 		(property "Description" "Mounting Hole without connection"
-			(at 266.7 143.51 0)
+			(at 261.62 160.02 0)
 			(effects
 				(font
@@
 	)
 	(symbol
-		(lib_id "Mechanical:MountingHole")
-		(at 266.7 158.75 0)
-		(unit 1)
-		(exclude_from_sim yes)
-		(in_bom no)
-		(on_board yes)
-		(dnp no)
-		(fields_autoplaced yes)
-		(property "Reference" "H4"
-			(at 269.24 157.4799 0)
-			(effects
-				(font
-					(size 1.27 1.27)
-				)
-				(justify left)
-			)
-		)
-		(property "Value" "MountingHole"
-			(at 269.24 160.0199 0)
-			(effects
-				(font
-					(size 1.27 1.27)
-				)
-				(justify left)
-			)
-		)
-		(property "Footprint" "MountingHole:MountingHole_2mm"
-			(at 266.7 158.75 0)
-			(effects
-				(font
-					(size 1.27 1.27)
-				)
-				(hide yes)
-			)
-		)
-		(property "Datasheet" "~"
-			(at 266.7 158.75 0)
-			(effects
-				(font
-					(size 1.27 1.27)
-				)
-				(hide yes)
-			)
-		)
-		(property "Description" "Mounting Hole without connection"
-			(at 266.7 158.75 0)
-			(effects
-				(font
-					(size 1.27 1.27)
-				)
-				(hide yes)
-			)
-		)
-		(instances
-			(project "VintageRadio"
-				(path "/7fa8ac5a-a2bc-40af-b61f-bda00e608227"
-					(reference "H4")
-					(unit 1)
-				)
-			)
-		)
-	)
-	(symbol
 		(lib_id "Device:R")
 		(at 138.43 69.85 0)
@@
 	(symbol
 		(lib_id "Mechanical:MountingHole")
-		(at 266.7 153.67 0)
-		(unit 1)
-		(exclude_from_sim yes)
-		(in_bom no)
-		(on_board yes)
-		(dnp no)
-		(fields_autoplaced yes)
-		(property "Reference" "H3"
-			(at 269.24 152.3999 0)
-			(effects
-				(font
-					(size 1.27 1.27)
-				)
-				(justify left)
-			)
-		)
-		(property "Value" "MountingHole"
-			(at 269.24 154.9399 0)
-			(effects
-				(font
-					(size 1.27 1.27)
-				)
-				(justify left)
-			)
-		)
-		(property "Footprint" "MountingHole:MountingHole_2mm"
-			(at 266.7 153.67 0)
-			(effects
-				(font
-					(size 1.27 1.27)
-				)
-				(hide yes)
-			)
-		)
-		(property "Datasheet" "~"
-			(at 266.7 153.67 0)
-			(effects
-				(font
-					(size 1.27 1.27)
-				)
-				(hide yes)
-			)
-		)
-		(property "Description" "Mounting Hole without connection"
-			(at 266.7 153.67 0)
-			(effects
-				(font
-					(size 1.27 1.27)
-				)
-				(hide yes)
-			)
-		)
-		(instances
-			(project "VintageRadio"
-				(path "/7fa8ac5a-a2bc-40af-b61f-bda00e608227"
-					(reference "H3")
-					(unit 1)
-				)
-			)
-		)
-	)
-	(symbol
-		(lib_id "Mechanical:MountingHole")
-		(at 266.7 148.59 0)
+		(at 266.7 160.02 0)
 		(unit 1)
 		(exclude_from_sim yes)
@@
 		(fields_autoplaced yes)
 		(property "Reference" "H2"
-			(at 269.24 147.3199 0)
+			(at 269.24 158.7499 0)
 			(effects
 				(font
@@
 		)
 		(property "Value" "MountingHole"
-			(at 269.24 149.8599 0)
+			(at 269.24 161.2899 0)
 			(effects
 				(font
@@
 		)
 		(property "Footprint" "MountingHole:MountingHole_2mm"
-			(at 266.7 148.59 0)
+			(at 266.7 160.02 0)
 			(effects
 				(font
@@
 		)
 		(property "Datasheet" "~"
-			(at 266.7 148.59 0)
+			(at 266.7 160.02 0)
 			(effects
 				(font
@@
 		)
 		(property "Description" "Mounting Hole without connection"
-			(at 266.7 148.59 0)
-			(effects
-				(font
+			(at 266.7 160.02 0)
+			(effects
+				(font
